File: pcb/esp32dev.kicad_pcb (KiCad board)
At the start: 2 copper layers, 1 part, among them U1 ESP32-C3

Commit message: Hmmmm
Parts:
- added AE1: PCB_Antenna, esp32dev:Texas_SWRA117D_2.4GHz_Left, F.Cu at (107.3, 87.8)
- added C1: 10uF, Capacitor_SMD:C_0805_2012Metric, F.Cu at (137.2, 95.9)
- added C2: 10uF, Capacitor_SMD:C_0805_2012Metric, F.Cu at (134.6, 95.9)
- added C3: 100nF, Capacitor_SMD:C_0402_1005Metric, F.Cu at (111.8, 87.6)
- added C4: 100nF, Capacitor_SMD:C_0402_1005Metric, F.Cu at (109.2, 87.6)
- added C5: 100nF, Capacitor_SMD:C_0402_1005Metric, F.Cu at (115.6, 87.6)
- added C6: 100nF, Capacitor_SMD:C_0402_1005Metric, F.Cu at (109.2, 90.8)
- added C7: 100nF, Capacitor_SMD:C_0402_1005Metric, F.Cu at (109.2, 96.5)
- added C8: 100nF, Capacitor_SMD:C_0402_1005Metric, F.Cu at (118.7, 87.6)
- added C9: 100nF, Capacitor_SMD:C_0402_1005Metric, F.Cu at (116.2, 96.5)
- added J1: ~, Connector_PinHeader_2.54mm:PinHeader_1x10_P2.54mm_Vertical, B.Cu at (111.1, 100.3)
- added J2: ~, Connector_PinHeader_2.54mm:PinHeader_1x10_P2.54mm_Vertical, B.Cu at (111.8, 85.1)
- added R1: 10k, Resistor_SMD:R_0603_1608Metric, F.Cu at (109.2, 93.3)
- added U2: AP1117-33, Package_TO_SOT_SMD:SOT-223-3_TabPin2, F.Cu at (128.9, 94.6)
- added U3: W25Q128JVS, Package_SO:SOIC-8_5.23x5.23mm_P1.27mm, F.Cu at (120.7, 93.3)
- U1: footprint Package_DFN_QFN:QFN-32-1EP_5x5mm_P0.5mm_EP3.1x3.1mm -> esp32dev:QFN-32-1EP_5x5mm_P0.5mm_EP3.1x3.1mm_ThermalVias
- moved U1 13.7 mm to (113.7, 92.1)
Connections:
- U1 pad 11: Net-(U1-Pad11) -> +3V3
- U1 pad 17: Net-(U1-Pad17) -> +3V3
- U1 pad 18: Net-(U1-Pad18) -> VDD_SPI
- U1 pad 19: Net-(U1-Pad19) -> F_RST
- U1 pad 2: Net-(U1-Pad2) -> +3V3
- U1 pad 20: Net-(U1-Pad20) -> F_WP
- U1 pad 21: Net-(U1-Pad21) -> F_CS
- U1 pad 22: Net-(U1-Pad22) -> F_CK
- U1 pad 23: Net-(U1-Pad23) -> F_DI
- U1 pad 24: Net-(U1-Pad24) -> F_DO
- U1 pad 3: Net-(U1-Pad3) -> +3V3
- U1 pad 31: Net-(U1-Pad31) -> +3V3
- U1 pad 32: Net-(U1-Pad32) -> +3V3
- U1 pad 33: Net-(U1-Pad33) -> GND
- U1 pad 7: Net-(U1-Pad7) -> EN
Routing:
- net +3V3: track 0.00 -> 9.00 mm, vias 0 -> 6
- net VBUS: track 0.00 -> 6.19 mm
- added copper zone on F.Cu, net +3V3
- added copper zone on In1.Cu, net +3V3
- added copper zone on B.Cu, net GND
- added copper zone on F.Cu, net GND
- added copper zone on In2.Cu, net GND
Other:
- board outline added: 38.1 x 20.3 mm
- copper layers 2 -> 4
- net class Default: clearance 0.2 -> 0.1524; trace_width 0.25 -> 0.1524; via_dia 0.8 -> 0.7; via_drill 0.4 -> 0.35
- rule trace_clearance: 0.2 -> 0.1524
- rule trace_min: 0.2 -> 0.1524

Commit message: Hmmmm
Parts:
- added C10: 10pF, Capacitor_SMD:C_0402_1005Metric, F.Cu at (116.8, 88.9)
- added C11: 10pF, Capacitor_SMD:C_0402_1005Metric, F.Cu at (110.5, 88.9)
- added D1: ~, Diode_SMD:D_SOD-123, F.Cu at (139.7, 100.3)
- added J3: USB-C, esp32dev:USB_C_Receptacle_HRO_TYPE-C-31-M-12, F.Cu at (145.4, 92.7)
- added R2: 22R, Resistor_SMD:R_0402_1005Metric, F.Cu at (137.2, 92.1)
- added R3: 22R, Resistor_SMD:R_0402_1005Metric, F.Cu at (137.2, 90.8)
- added R4: 1.5k, Resistor_SMD:R_0402_1005Metric, F.Cu at (137.2, 88.3)
- added R5: 5.1k, Resistor_SMD:R_0402_1005Metric, F.Cu at (137.2, 89.5)
- added R6: 5.1k, Resistor_SMD:R_0402_1005Metric, F.Cu at (137.2, 93.3)
- added Y1: ~, Crystal:Crystal_SMD_3225-4Pin_3.2x2.5mm, F.Cu at (113.7, 88.9)
- AE1: value PCB_Antenna -> ~
- moved C5 5.72 mm to (121.3, 87.6)
- moved C3 2.84 mm to (109.2, 86.4), turned to 180 degrees
- moved U1 1.91 mm to (113.7, 94.0)
- moved C9 1.42 mm to (116.8, 97.8)
- moved C7 1.27 mm to (109.2, 97.8)
- moved U3 0.90 mm to (121.3, 94.0)
Connections:
- U1 pad 25: Net-(U1-Pad25) -> DM
- U1 pad 26: Net-(U1-Pad26) -> DP
Other:
- board size 38.1 x 20.3 mm -> 47.6 x 20.3 mm

Commit message: Hmmm
Parts:
- removed R4: 1.5k, Resistor_SMD:R_0402_1005Metric
- added C12: NM, Capacitor_SMD:C_0603_1608Metric, F.Cu at (109.2, 97.8)
- added C13: NM, Capacitor_SMD:C_0603_1608Metric, F.Cu at (109.2, 94.0)
- added C14: 100nF, Capacitor_SMD:C_0402_1005Metric, F.Cu at (113.0, 94.6)
- added D2: WS2812C-2020, esp32dev:LED_WS2812C-2020, F.Cu at (134.0, 95.9)
- added L1: L, Inductor_SMD:L_0603_1608Metric, F.Cu at (109.2, 95.9)
- added SW1: ~, esp32dev:TS-1088R-02526, F.Cu at (146.1, 102.9)
- added SW2: ~, esp32dev:TS-1088R-02526, F.Cu at (139.7, 102.9)
- AE1: footprint esp32dev:Texas_SWRA117D_2.4GHz_Left -> esp32dev:Texas_SWRA117D_2.4GHz_Right
- J1, J2: footprint Connector_PinHeader_2.54mm:PinHeader_1x10_P2.54mm_Vertical -> Connector_PinHeader_2.54mm:PinHeader_2x10_P2.54mm_Vertical
- R1: footprint Resistor_SMD:R_0603_1608Metric -> Resistor_SMD:R_0402_1005Metric
- Y1: value ~ -> 40MHz
- moved C1 16.8 mm to (147.3, 82.5), turned to 90 degrees
- moved U2 16.3 mm to (141.6, 84.5)
- moved D1 14.8 mm to (147.3, 87.6), turned to 270 degrees
- moved C3 12.3 mm to (116.2, 96.5)
- moved U3 11.4 mm to (132.1, 90.2), turned to 180 degrees
- moved C4 10.3 mm to (116.2, 95.2)
- moved C2 9.92 mm to (142.2, 89.5), turned to 0 degrees
- moved C8 8.82 mm to (126.4, 92.1), turned to 270 degrees
- moved AE1 8.06 mm to (107.3, 95.9)
- moved R5 6.63 mm to (139.1, 95.9)
- moved R2 6.63 mm to (139.1, 98.4)
- moved R3 6.63 mm to (139.1, 97.2)
- moved R6 6.63 mm to (139.1, 99.7)
- moved C9 5.85 mm to (122.6, 96.5)
- moved U1 5.85 mm to (119.4, 92.7), turned to 45 degrees
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Connections:
- net F_RST renamed IO12_F_RST
- net F_WP renamed IO13_F_WP
- net Net-(U1-Pad10) renamed IO5_MTDI
- net Net-(U1-Pad12) renamed IO6_MTCK
- net Net-(U1-Pad13) renamed IO7_MTDO
- net Net-(U1-Pad14) renamed IO8
- net Net-(U1-Pad15) renamed IO9
- net Net-(U1-Pad16) renamed IO10
- net Net-(U1-Pad4) renamed IO0
- net Net-(U1-Pad5) renamed IO1
- net Net-(U1-Pad6) renamed IO2
- net Net-(U1-Pad8) renamed IO3
- net Net-(U1-Pad9) renamed IO4_MTMS
- J1 pad 2: Net-(J1-Pad2) -> Net-(J1-Pad1)
- J1 pad 4: Net-(J1-Pad4) -> Net-(J1-Pad3)
- J1 pad 6: Net-(J1-Pad6) -> Net-(J1-Pad5)
- J1 pad 8: Net-(J1-Pad8) -> Net-(J1-Pad7)
- J1 pad 9: Net-(J1-Pad9) -> Net-(J1-Pad10)
- J2 pad 2: Net-(J2-Pad2) -> Net-(J2-Pad1)
- J2 pad 4: Net-(J2-Pad4) -> Net-(J2-Pad3)
- J2 pad 6: Net-(J2-Pad6) -> Net-(J2-Pad5)
- J2 pad 8: Net-(J2-Pad8) -> Net-(J2-Pad7)
- J2 pad 9: Net-(J2-Pad9) -> Net-(J2-Pad10)
- R2 pad 2: DM -> IO18_DM
- R3 pad 2: DP -> IO19_DP
- U1 pad 1: Net-(AE1-Pad1) -> Net-(C13-Pad1)
- U1 pad 25: DM -> IO18_DM
- U1 pad 26: DP -> IO19_DP
- U1 pad 27: Net-(U1-Pad27) -> IO20_U0RX
- U1 pad 28: Net-(U1-Pad28) -> IO21_U0TX
Routing:
- net F_CS: track 0.00 -> 17.4 mm, vias 0 -> 2
- net IO13_F_WP: track 0.00 -> 15.1 mm
- net F_DI: track 0.00 -> 10.4 mm
- net F_CK: track 0.00 -> 9.87 mm
- net +3V3: track 9.00 -> 0.00 mm, vias 6 -> 0
- net IO12_F_RST: track 0.00 -> 7.14 mm
- net VDD_SPI: track 0.00 -> 6.81 mm
- net VBUS: track 6.19 -> 0.00 mm
- net Net-(J2-Pad7): track 0.00 -> 2.54 mm
- net Net-(J2-Pad5): track 0.00 -> 2.54 mm
- net Net-(J2-Pad3): track 0.00 -> 2.54 mm
- net Net-(J2-Pad19): track 0.00 -> 2.54 mm
- net Net-(J2-Pad17): track 0.00 -> 2.54 mm
- net Net-(J2-Pad15): track 0.00 -> 2.54 mm
- net Net-(J2-Pad10): track 0.00 -> 2.54 mm
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- removed copper zone on F.Cu, net +3V3
Other:
- board size 47.6 x 20.3 mm -> 47.6 x 25.4 mm

Commit message: Hmmmm
Parts:
- D2: value WS2812C-2020 -> WS2812
- L1: value L -> 0R
- moved C14 5.99 mm to (118.1, 97.8), turned to 0 degrees
- moved R1 3.70 mm to (116.2, 97.8)
- moved C4 3.17 mm to (113.0, 95.2)
- moved Y1 2.01 mm to (112.4, 89.5)
- moved C10 1.91 mm to (109.9, 88.3)
- moved C11 1.91 mm to (109.9, 90.2)
- moved C6 0.64 mm to (113.0, 92.7)
- moved R2 0.63 mm to (138.4, 98.4)
- moved R3 0.63 mm to (138.4, 97.2)
- moved R5 0.63 mm to (138.4, 95.9)
- moved R6 0.63 mm to (138.4, 99.7)
Connections:
- D2 pad 2: Net-(D2-Pad2) -> GND
- D2 pad 4: Net-(D2-Pad4) -> +3V3
- J1 pad 15: IO19_DP -> Net-(J1-Pad15)
- J1 pad 16: IO19_DP -> Net-(J1-Pad15)
- J1 pad 17: IO18_DM -> Net-(J1-Pad17)
- J1 pad 18: IO18_DM -> Net-(J1-Pad17)
- J2 pad 10: Net-(J2-Pad10) -> IO18_DM
- J2 pad 11: IO21_U0TX -> Net-(J2-Pad11)
- J2 pad 12: IO21_U0TX -> Net-(J2-Pad11)
- J2 pad 13: IO20_U0RX -> Net-(J2-Pad13)
- J2 pad 14: IO20_U0RX -> Net-(J2-Pad13)
- J2 pad 3: Net-(J2-Pad3) -> IO21_U0TX
- J2 pad 4: Net-(J2-Pad3) -> IO21_U0TX
- J2 pad 5: Net-(J2-Pad5) -> IO20_U0RX
- J2 pad 6: Net-(J2-Pad5) -> IO20_U0RX
- J2 pad 7: Net-(J2-Pad7) -> IO19_DP
- J2 pad 8: Net-(J2-Pad7) -> IO19_DP
- J2 pad 9: Net-(J2-Pad10) -> IO18_DM
- U1 pad 20: IO13_F_WP -> F_CS
- U1 pad 21: F_CS -> F_CK
- U1 pad 22: F_CK -> F_DI
- U1 pad 23: F_DI -> F_DO
- U1 pad 24: F_DO -> Net-(U1-Pad24)
Routing:
- net F_DO: track 0.00 -> 17.9 mm, vias 0 -> 2
- net +5V: track 0.00 -> 16.4 mm
- net IO19_DP: track 2.54 -> 14.8 mm
- net IO18_DM: track 2.54 -> 11.7 mm
- net Net-(C13-Pad1): track 0.00 -> 8.66 mm
- net Net-(J3-PadA7): track 0.00 -> 8.11 mm
- net Net-(C10-Pad1): track 0.00 -> 7.06 mm
- net +3V3: track 0.00 -> 6.30 mm, vias 0 -> 1
- net Net-(J3-PadA6): track 0.00 -> 5.79 mm
- net Net-(C11-Pad1): track 0.00 -> 4.25 mm
- net Net-(J3-PadA5): track 0.00 -> 4.07 mm
- net Net-(J3-PadB5): track 0.00 -> 3.76 mm
- net Net-(AE1-Pad1): track 0.00 -> 3.03 mm
- net Net-(J2-Pad7): track 2.54 -> 0.00 mm
- net Net-(J2-Pad5): track 2.54 -> 0.00 mm
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Other:
- board text added: "Esp32Dev, rev. a ESP32-C3 Dev Board (C) 2021 Lars Boegild Thomsen"
