File: pcb/esp32dev.sch (KiCad schematic (older format))
At the start: 1 part, among them U1 ESP32-C3

Commit message: Hmmmm
Parts:
- added AE1: PCB_Antenna, esp32dev:Texas_SWRA117D_2.4GHz_Left, symbol esp32dev:PCB_Antenna
- added C1, C2: 10uF, Capacitor_SMD:C_0805_2012Metric, symbol Device:C
- added C3, C4, C5, C6, C7, C8, C9: 100nF, Capacitor_SMD:C_0402_1005Metric, symbol Device:C
- added J1, J2: ~, Connector_PinHeader_2.54mm:PinHeader_1x10_P2.54mm_Vertical, symbol Connector_Generic:Conn_01x10
- added R1: 10k, Resistor_SMD:R_0603_1608Metric, symbol Device:R
- added U2: AP1117-33, Package_TO_SOT_SMD:SOT-223-3_TabPin2, symbol Regulator_Linear:AP1117-33
- added U3: W25Q128JVS, Package_SO:SOIC-8_5.23x5.23mm_P1.27mm, symbol Memory_Flash:W25Q128JVS
- U1: footprint Package_DFN_QFN:QFN-32-1EP_5x5mm_P0.5mm_EP3.1x3.1mm -> esp32dev:QFN-32-1EP_5x5mm_P0.5mm_EP3.1x3.1mm_ThermalVias
Connections:
- net labels added: +3.3V, EN, F_CK, F_CS, F_DI, F_DO, F_RST, F_WP, GND, VBUS, VDD_SPI
- wire segments 0 -> 76

Commit message: Hmmmm
Parts:
- added C10, C11: 10pF, Capacitor_SMD:C_0402_1005Metric, symbol Device:C
- added D1: ~, Diode_SMD:D_SOD-123, symbol Device:D_Schottky
- added J3: USB-C, esp32dev:USB_C_Receptacle_HRO_TYPE-C-31-M-12, symbol esp32dev:USB_C_Receptacle_USB2.0
- added R2, R3: 22R, Resistor_SMD:R_0402_1005Metric, symbol Device:R
- added R4: 1.5k, Resistor_SMD:R_0402_1005Metric, symbol Device:R
- added R5, R6: 5.1k, Resistor_SMD:R_0402_1005Metric, symbol Device:R
- added Y1: ~, Crystal:Crystal_SMD_3225-4Pin_3.2x2.5mm, symbol Device:Crystal_GND24
- AE1: value PCB_Antenna -> ~
Connections:
- net labels added: +5V, DM, DP
- wire segments 76 -> 124
- no-connect marks 0 -> 2

Commit message: Hmmm
Parts:
- removed J1, J2: ~, Connector_PinHeader_2.54mm:PinHeader_1x10_P2.54mm_Vertical, symbol Connector_Generic:Conn_01x10
- removed R4: 1.5k, Resistor_SMD:R_0402_1005Metric, symbol Device:R
- added C12, C13: NM, Capacitor_SMD:C_0603_1608Metric, symbol Device:C
- added C14: 100nF, Capacitor_SMD:C_0402_1005Metric, symbol Device:C
- added D2: WS2812C-2020, esp32dev:LED_WS2812C-2020, symbol esp32dev:WS2812C-2020
- added J1, J2: ~, Connector_PinHeader_2.54mm:PinHeader_2x10_P2.54mm_Vertical, symbol Connector_Generic:Conn_02x10_Odd_Even
- added L1: L, Inductor_SMD:L_0603_1608Metric, symbol Device:L
- added SW1, SW2: ~, esp32dev:TS-1088R-02526, symbol esp32dev:SW_Push
- AE1: footprint esp32dev:Texas_SWRA117D_2.4GHz_Left -> esp32dev:Texas_SWRA117D_2.4GHz_Right
- R1: footprint Resistor_SMD:R_0603_1608Metric -> Resistor_SMD:R_0402_1005Metric; LCSC (none) -> C25744
- Y1: value ~ -> 40MHz
Connections:
- net labels added: IO0, IO1, IO10, IO12_F_RST, IO13_F_WP, IO18_DM, IO19_DP, IO2, IO20_U0RX, IO21_U0TX, IO3, IO4_MTMS, IO5_MTDI, IO6_MTCK, IO7_MTDO, IO8, IO9
- net labels removed: DM, DP, F_RST, F_WP
- wire segments 124 -> 173

Commit message: Hmmmm
Parts:
- D2: value WS2812C-2020 -> WS2812
- L1: value L -> 0R; LCSC (none) -> C21189
- U1: symbol esp32dev:ESP32-C3 -> esp32dev-rescue:ESP32-C3-esp32dev
Connections:
- wire segments 173 -> 175
Changed lines of the file:
@@
 $EndDescr
 $Comp
-L esp32dev:ESP32-C3 U1
+L esp32dev-rescue:ESP32-C3-esp32dev U1
 U 1 1 618A9FF1
 P 9300 1900
@@
 U 1 1 61A4E43A
 P 7950 2900
-F 0 "L1" V 8050 3000 50  0000 C CNN
-F 1 "L" V 8050 2800 50  0000 C CNN
+F 0 "L1" V 8000 3050 50  0000 C CNN
+F 1 "0R" V 8000 2750 50  0000 C CNN
 F 2 "Inductor_SMD:L_0603_1608Metric" H 7950 2900 50  0001 C CNN
 F 3 "~" H 7950 2900 50  0001 C CNN
+F 4 "C21189" V 7950 2900 50  0001 C CNN "LCSC"
 	1    7950 2900
 	0    -1   -1   0
@@
 Text GLabel 2800 4050 2    50   Input ~ 0
 IO19_DP
-Text GLabel 9900 4750 0    50   Input ~ 0
+Text GLabel 9900 5600 0    50   Input ~ 0
 IO18_DM
-Text GLabel 9900 4650 0    50   Input ~ 0
+Text GLabel 9900 5500 0    50   Input ~ 0
 IO19_DP
 Wire Wire Line
-	9900 4650 10200 4650
-Wire Wire Line
-	10200 4750 9900 4750
+	9900 5500 10200 5500
+Wire Wire Line
+	10200 5600 9900 5600
 Text GLabel 10200 1100 2    50   Input ~ 0
 IO2
@@
 Wire Wire Line
 	10200 1100 10100 1100
-Text GLabel 9900 5800 0    50   Input ~ 0
+Text GLabel 9900 5400 0    50   Input ~ 0
 IO20_U0RX
-Text GLabel 9900 5700 0    50   Input ~ 0
+Text GLabel 9900 5300 0    50   Input ~ 0
 IO21_U0TX
 Wire Wire Line
-	9900 5700 10200 5700
-Wire Wire Line
-	10200 5800 9900 5800
+	9900 5300 10200 5300
+Wire Wire Line
+	10200 5400 9900 5400
 Text GLabel 2550 6700 2    50   Input ~ 0
 IO12_F_RST
@@
 Wire Wire Line
 	10700 5700 10200 5700
-Connection ~ 10200 5700
 Wire Wire Line
 	10200 5800 10700 5800
-Connection ~ 10200 5800
 Wire Wire Line
 	10700 5900 10200 5900
@@
 Wire Wire Line
 	10700 6100 10200 6100
-Connection ~ 10200 4650
-Connection ~ 10200 4750
 $Comp
 L esp32dev:WS2812C-2020 D2
 U 1 1 61BF2B33
 P 5250 6000
-F 0 "D2" H 5594 6046 50  0000 L CNN
-F 1 "WS2812C-2020" H 5594 5955 50  0000 L CNN
+F 0 "D2" H 5050 6250 50  0000 L CNN
+F 1 "WS2812" H 5300 6250 50  0000 L CNN
 F 2 "esp32dev:LED_WS2812C-2020" H 5300 5700 50  0001 L TNN
 F 3 "https://ipfs-pin.com/ipfs/QmUrWWQTAtUDvCNqULeBaKaw2HwTcne6zNz3L68ZhahRnx/WS2812C-2020_361_V1.0_EN_20031610354448.pdf" H 5350 5625 50  0001 L TNN
@@
 	1    0    0    -1
 $EndComp
+$Comp
+L power:+3.3V #PWR0120
+U 1 1 619AD6B1
+P 5250 5600
+F 0 "#PWR0120" H 5250 5450 50  0001 C CNN
+F 1 "+3.3V" H 5265 5773 50  0000 C CNN
+F 2 "" H 5250 5600 50  0001 C CNN
+F 3 "" H 5250 5600 50  0001 C CNN
+	1    5250 5600
+	1    0    0    -1
+$EndComp
+$Comp
+L power:GND #PWR0124
+U 1 1 619AE4A4
+P 5250 6400
+F 0 "#PWR0124" H 5250 6150 50  0001 C CNN
+F 1 "GND" H 5255 6227 50  0000 C CNN
+F 2 "" H 5250 6400 50  0001 C CNN
+F 3 "" H 5250 6400 50  0001 C CNN
+	1    5250 6400
+	1    0    0    -1
+$EndComp
+Wire Wire Line
+	5250 6400 5250 6300
+Wire Wire Line
+	5250 5600 5250 5700
+Connection ~ 10200 5300
+Connection ~ 10200 5400
+Connection ~ 10200 5500
+Connection ~ 10200 5600
 $EndSCHEMATC
